File: PCB/finalboard/finalboard.kicad_sch (KiCad schematic)
At the start: 27 parts, among them J1 USB_C_Receptacle_USB2.0, J2 Conn_01x02, J3 Conn_01x04, J6 AudioJack4, Q1 MMDT3904, U1 ESP32-S3-WROOM-1, U3 USBLC6-2SC6, U5 SN74LVC1T45DRL, U6 SN74LVC1T45DRL, U7 AMS1117-3.3, U8 MCP73831-2-OT

Commit message: Incorporated Feedback
Parts:
- removed Q1: MMDT3904, Package_TO_SOT_SMD:SOT-363_SC-70-6, symbol Transistor_BJT:MMDT3904
- removed TP2: TestPoint, TestPoint:TestPoint_Pad_D4.0mm, symbol Connector:TestPoint
- added C4, C5: 10u, Capacitor_SMD:C_1206_3216Metric, symbol Device:C
- added C6: 0.1u, Capacitor_SMD:C_1206_3216Metric, symbol Device:C
- added D4: GREEN, LED_SMD:LED_1206_3216Metric, symbol Device:LED
- added D5: YELLOW, LED_SMD:LED_1206_3216Metric, symbol Device:LED
- added D6: 1N5822, Diode_THT:D_DO-201AD_P15.24mm_Horizontal, symbol Diode:1N5822
- added D7: BLUE, LED_SMD:LED_1206_3216Metric, symbol Device:LED
- added J4, J7: Conn_01x04, Connector_PinHeader_2.54mm:PinHeader_1x04_P2.54mm_Vertical, symbol Connector_Generic:Conn_01x04
- added J5: Conn_01x02, Connector_PinHeader_2.54mm:PinHeader_1x02_P2.54mm_Vertical, symbol Connector_Generic:Conn_01x02
- added Q1: DMG2301L, Package_TO_SOT_SMD:SOT-23, symbol Transistor_FET:DMG2301L
- added Q3: S8550, Package_TO_SOT_THT:TO-92_Inline, symbol Transistor_BJT:S8550
- added R10, R11, R12, R16: 10k, Resistor_SMD:R_1206_3216Metric, symbol Device:R
- added R13, R17: 100k, Resistor_SMD:R_1206_3216Metric, symbol Device:R
- added R15: 6.8k, Resistor_SMD:R_1206_3216Metric, symbol Device:R
- added R6: 220, Resistor_SMD:R_1206_3216Metric, symbol Device:R
- added R7: 1000, Resistor_SMD:R_1206_3216Metric, symbol Device:R
- added R8: 4.7k, Resistor_SMD:R_1206_3216Metric, symbol Device:R
- added R9: 470, Resistor_SMD:R_1206_3216Metric, symbol Device:R
- added SW1, SW3: SW_DIP_x01, symbol Switch:SW_DIP_x01
- added U10, U9: SN74LVC1T45DRL, Package_TO_SOT_SMD:SOT-563, symbol Logic_LevelTranslator:SN74LVC1T45DRL
- added U11: MCP23008-xSO, Package_SO:SOIC-18W_7.5x11.6mm_P1.27mm, symbol Interface_Expansion:MCP23008-xSO
- D1: value LED -> RED
- D2: value LED -> BLUE
- D3: value LED -> YELLOW
- R3, R4, R5: value R -> 470
Connections:
- net PWR_TRAN_LCD is gone; now on net LED_BACKLIGHT: U1.39 (GPIO1/TOUCH1/ADC1_CH0)
- net PWR_TRAN_TFT is gone; now on net LCD_DC: U1.38 (GPIO2/TOUCH2/ADC1_CH1)
- net +3V3: now also U2.1 (VCC), C4.1, C5.1, J4.4 (Pin_4), R10.1, R11.1, R17.1, R6.1, U10.1 (VCCA), U11.18 (VDD), U11.3 (A2), U11.4 (A1), U9.1 (VCCA), U9.5 (DIR)
- net ESP_RX0: now also R9.2
- net ESP_RX2: now also U10.3 (A); no longer J3.3 (Pin_3)
- net ESP_SS_RX0: now also R4.2; no longer U4.4 (TX0)
- net ESP_SS_TX0: now also R3.2; no longer U4.3 (RXD)
- net ESP_TX0: now also R5.2
- net ESP_TX2: now also U9.3 (A); no longer J3.2 (Pin_2)
- net GND: now also D1.1 (K), D2.1 (K), D3.1 (K), J2.2 (Pin_2), U8.2 (V_{SS}), C4.2, C5.2, C6.1, D7.1 (K), J4.1 (Pin_1), J5.1 (Pin_1), Q3.3 (C), R13.2, R16.1, R8.2, SW1.2, U10.2 (GND), U10.5 (DIR), U11.5 (A0), U11.9 (VSS), U9.2 (GND); no longer R3.1, R4.1, R5.1
- net RECORDING_LED: now reaches D1.2 (A)
- net RECORDING_LED: now also U11.11 (GP1); no longer U1.12 (GPIO8/TOUCH8/ADC1_CH7/SUBSPICS1)
- net SCL: now reaches U1.17 (GPIO9/TOUCH9/ADC1_CH8/FSPIHD/SUBSPIHD)
- net SCL: now also R11.2, U11.1 (SCL); no longer D2.2 (A)
- net at U1.27 (GPIO0/BOOT): now also J5.2 (Pin_2)
- net at U1.3 (EN): now also C6.2, R12.1, R17.2
- net LED_BUILTIN: now reaches U1.31 (GPIO38/FSPIWP/SUBSPIWP)
- net LED_BUILTIN: now also D7.2 (A); no longer D3.2 (A)
- net at U1.32 (MTCK/GPIO39/CLK_OUT3/SUBSPICS1): now also J7.4 (Pin_4)
- net at U1.33 (MTDO/GPIO40/CLK_OUT2): now also J7.3 (Pin_3)
- net at U1.34 (MTDI/GPIO41/CLK_OUT1): now also J7.2 (Pin_2)
- net at U1.35 (MTMS/GPIO42): now also J7.1 (Pin_1)
- net ADC_Battery: now reaches U1.4 (GPIO4/TOUCH4/ADC1_CH3)
- net ADC_Battery: now also R15.1, R16.2
- net LCD_DC: now reaches U2.5 (DC/RS)
- net LED_BACKLIGHT: now reaches U2.8 (LED)
- net at U8.1 (STAT): now also D5.1 (K)
- net VBAT: now reaches U8.3 (V_{BAT})
- net VBAT: now also J2.1 (Pin_1), Q1.3 (D), R15.2
- net VBUS: now reaches U8.4 (V_{DD})
- net VBUS: now also J1.A4 (VBUS), J1.A9 (VBUS), J1.B4 (VBUS), J1.B9 (VBUS), U3.5 (VBUS), D5.2 (A), D6.2 (A), Q1.1 (G), R13.1
- net at U8.5 (PROG): now also R8.1
- net CA_RX: now reaches J6.R1, U5.4 (B)
- net CA_5V: now reaches J6.R2, U5.6 (VCCB), U6.6 (VCCB)
- net CA_TX: now reaches J6.T, U6.4 (B)
- net at U4.5 (PPS): now also R7.2
- net BMS_RX: now reaches J3.1 (Pin_1)
- net BMS_RX: now also U9.4 (B)
- new net: Q3.2 (B), R7.1
- new net: D6.1 (K), Q1.2 (S), SW3.1
- new net: J4.3 (Pin_3), R9.1
- new net: R12.2, SW1.1
- new net: D4.1 (K), Q3.1 (E)
- new net: D4.2 (A), R6.2
- new net: J4.2 (Pin_2), R5.1
- new net: R3.1, U4.3 (RXD)
- new net: C1.1, SW3.2, U7.3 (VI)
- new net: R4.1, U4.4 (TX0)
- new net BMS_TX: J3.2 (Pin_2), U10.4 (B)
- new net BMS_VCC: J3.3 (Pin_3), U10.6 (VCCB), U9.6 (VCCB)
- new net SDA: R10.2, U1.12 (GPIO8/TOUCH8/ADC1_CH7/SUBSPICS1), U11.2 (SDA)
- new net SDCARD_LED: D3.2 (A), U11.10 (GP0)
- new net WIFI_LED: D2.2 (A), U11.12 (GP2)
- no-connect marks 6 -> 20
Other:
- note added: "10k = 0.1A 5k = 0.2A 2k = 0.5A 1k = 1.0A"
- note added: "ESP32 + IO Expander"
- note added: "GPS Module GPS NEO-6M"
- note added: "Hosyond 3.5 Inches TFT"
- note added: "JTAG"
- note added: "LIPO Charger and Battery Connector"
- note added: "Short to Enter Bootloader"
- note added: "Testpoints = Touch Buttons"
- note added: "UART Debug"
- note added: "UART to Cycle Analyst"
- note added: "UART to DalyBMS Battery"
- note added: "USB Protection + Regulator"
- moved on the sheet: C1, C2, C3, D1, D2, D3, J1, J2, J3, J6, R1, R2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

Commit message: Schematic Mostly Done
check esp32 pins
Parts:
- removed R6: 220, Resistor_SMD:R_1206_3216Metric, symbol Device:R
- removed U10, U5, U6, U9: SN74LVC1T45DRL, Package_TO_SOT_SMD:SOT-563, symbol Logic_LevelTranslator:SN74LVC1T45DRL
- added C10, C12, C13, C14, C15, C18, C22: 0.1u, Capacitor_SMD:C_0603_1608Metric, symbol Device:C
- added C11: 1u, Capacitor_SMD:C_1206_3216Metric, symbol Device:C
- added C16, C17, C20, C21: 10u, Capacitor_SMD:C_1206_3216Metric, symbol Device:C
- added C19: 0.1u, Capacitor_SMD:C_1206_3216Metric, symbol Device:C
- added C7, C9: 1u, Capacitor_SMD:C_0603_1608Metric, symbol Device:C
- added C8: 22u, Capacitor_SMD:C_0603_1608Metric, symbol Device:C
- added R14, R19, R20: 470, Resistor_SMD:R_1206_3216Metric, symbol Device:R
- added R18: 100, Resistor_SMD:R_1206_3216Metric, symbol Device:R
- added U12, U5: ~, symbol wc_sys_symbol:PI4ULS5V202UEX
- C1, C2, C5: value 10u -> 22u
- C4, C6: footprint Capacitor_SMD:C_1206_3216Metric -> Capacitor_SMD:C_0603_1608Metric
- R12: value 10k -> 470
- R17: value 100k -> 10K
- renumbered TP3 to TP2
Connections:
- net +3V3: now also D4.2 (A), C10.1, C11.1, C13.1, C14.1, C19.1, C7.1, C8.1, C9.1, U12.1 (VCCA), U12.5 (EN), U5.1 (VCCA), U5.5 (EN); no longer J4.4 (Pin_4)
- net BMS_RX: now also U5.7 (B1)
- net BMS_TX: now also C15.1, U5.6 (B2)
- net BMS_VCC: now also C17.1, U5.8 (VCCB)
- net CA_5V: now also C16.1, U12.8 (VCCB)
- net CA_RX: now also U12.7 (B1)
- net CA_TX: now also C18.1, U12.6 (B2)
- net ESP_RX1: now also U1.11 (GPIO18/U1RXD/ADC2_CH7/CLK_OUT3), R14.2; no longer U1.10 (GPIO17/U1TXD/ADC2_CH6)
- net ESP_RX2: now also U1.5 (GPIO5/TOUCH5/ADC1_CH4), R20.2; no longer U1.23 (GPIO21)
- net ESP_TX1: now also R12.2, U1.10 (GPIO17/U1TXD/ADC2_CH6); no longer U1.22 (GPIO14/TOUCH14/ADC2_CH3/FSPIWP/FSPIDQS/SUBSPIWP)
- net ESP_TX2: now also U1.4 (GPIO4/TOUCH4/ADC1_CH3), R19.2; no longer U1.11 (GPIO18/U1RXD/ADC2_CH7/CLK_OUT3)
- net GND: now also C10.2, C11.2, C12.1, C13.2, C14.2, C15.2, C16.2, C17.2, C18.2, C19.2, C20.2, C21.2, C22.1, C7.2, C8.2, C9.2, U12.4 (GND), U5.4 (GND)
- net LCD_DC: now also U1.25 (GPIO48/SPICLK_N/SUBSPICLK_N_DIFF); no longer U1.38 (GPIO2/TOUCH2/ADC1_CH1)
- net SCL: now also R10.2; no longer R11.2
- net SDA: now also R11.2; no longer R10.2
- net VBAT: now also C21.1
- net VBUS: now also C20.1
- net at C6.2, R17.2, U1.3 (EN): now also SW1.1; no longer R12.1
- net at TP1.1: now also U1.39 (GPIO1/TOUCH1/ADC1_CH0); no longer U1.15 (GPIO3/TOUCH3/ADC1_CH2)
- net LCD_BACKLIGHT: now reaches U1.24 (GPIO47/SPICLK_P/SUBSPICLK_P_DIFF)
- net LCD_BACKLIGHT: now also U2.8 (LED)
- net BOOT: now reaches J5.2 (Pin_2), U1.27 (GPIO0/BOOT)
- net at TP2.1: now also U1.38 (GPIO2/TOUCH2/ADC1_CH1); no longer U1.5 (GPIO5/TOUCH5/ADC1_CH4)
- net LCD_TIRQ: now reaches U1.8 (GPIO15/U0RTS/ADC2_CH4/XTAL_32K_P)
- net LCD_TIRQ: now also U2.14 (T_IRQ)
- net at U8.1 (STAT): now also R18.1; no longer D5.1 (K)
- net Vinput: now reaches C1.1, SW3.2, U7.3 (VI)
- net Vinput: now also C22.2
- net ADC_Battery renamed DIVIDED_VBAT
- net DIVIDED_VBAT: now also U1.15 (GPIO3/TOUCH3/ADC1_CH2), C12.2; no longer U1.4 (GPIO4/TOUCH4/ADC1_CH3)
- removed net LED_BACKLIGHT: U1.39 (GPIO1/TOUCH1/ADC1_CH0), U2.8 (LED)
- net SS1 renamed CS_SD
- net SS2 renamed CS_LCD
- net CS_LCD: now also U1.22 (GPIO14/TOUCH14/ADC2_CH3/FSPIWP/FSPIDQS/SUBSPIWP)
- net SS3 renamed CS_TOUCH
- net CS_TOUCH: now also U1.23 (GPIO21)
- new net: R14.1, U12.3 (A2)
- new net: R20.1, U5.3 (A2)
- new net: R12.1, U12.2 (A1)
- new net: R19.1, U5.2 (A1)
- new net: D5.1 (K), R18.2
- new net VCC: J4.4 (Pin_4)
- no-connect marks 20 -> 17
Other:
- note added: "Battery JST-PH Check Polarity"
- note added: "LIPO Charger + Divider"
- note added: "PI4ULS5V202UEX"
- note added: "Sleeve Ring2 Ring1 Tip"
- note removed: "LIPO Charger and Battery Connector"
- note removed: "Testpoints = Touch Buttons"
- moved on the sheet: C1, C2, C3, C5, C6, D1, D2, D3, D4, D7, J3, J4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

Commit message: Fixed Footprints, connected all nets
Parts:
- removed C13: 0.1u, Capacitor_SMD:C_0603_1608Metric, symbol Device:C
- removed C3: 10u, Capacitor_SMD:C_1206_3216Metric, symbol Device:C
- removed C7: 1u, Capacitor_SMD:C_0603_1608Metric, symbol Device:C
- removed R12, R14, R19, R20: 470, Resistor_SMD:R_1206_3216Metric, symbol Device:R
- added D7: 3.6V, Diode_SMD:D_MiniMELF, symbol Device:D_Zener
- added J5: Conn_02x06_Counter_Clockwise, Connector_PinSocket_2.54mm:PinSocket_2x06_P2.54mm_Vertical, symbol Connector_Generic:Conn_02x06_Counter_Clockwise
- C5: renamed from C1; value 22u -> 10u
- D1: renamed from D6; footprint Diode_THT:D_DO-201AD_P15.24mm_Horizontal -> Diode_SMD:D_SMA
- J2: renamed from J7; footprint Connector_PinHeader_2.54mm:PinHeader_1x04_P2.54mm_Vertical -> Connector_PinSocket_2.54mm:PinSocket_1x04_P2.54mm_Vertical
- J4: footprint Connector_PinHeader_2.54mm:PinHeader_1x04_P2.54mm_Vertical -> Connector_PinSocket_2.54mm:PinSocket_1x04_P2.54mm_Vertical
- Q2: renamed from Q3; footprint Package_TO_SOT_THT:TO-92_Inline -> Package_TO_SOT_SMD:SOT-23
- R19: renamed from R7; value 1000 -> 1k
- SW1: footprint (none) -> Button_Switch_THT:SW_PUSH_6mm_H5mm
- SW2: renamed from SW3; footprint (none) -> Button_Switch_THT:Push_E-Switch_KS01Q01
- U6: renamed from U12; value ~ -> PI4ULS5V202; footprint (none) -> wc_sys_footprint:PI4ULS5V202UEX; symbol wc_sys_symbol:PI4ULS5V202UEX -> wc_sys_symbol:PI4ULS5V202
- U7: renamed from U5; value ~ -> PI4ULS5V202; footprint (none) -> wc_sys_footprint:PI4ULS5V202UEX; symbol wc_sys_symbol:PI4ULS5V202UEX -> wc_sys_symbol:PI4ULS5V202
- U8: renamed from U2; footprint wc_sys_footprint:LCD3.5tft -> wc_sys_footprint:3.5_inch_SPI_Module_ILI9488; symbol wc_sys_symbol:LCD3.5 -> wc_sys_symbol:3.5inch_SPI Display_MSP3520
- U9: renamed from U4; footprint wc_sys_footprint:NEO-6M -> wc_sys_footprint:GT-U7
- renumbered C6 to C1, C21 to C10, C12 to C11, C17 to C12, C16 to C13, C15 to C14, C18 to C15, C14 to C16, C11 to C17, C5 to C18, C4 to C19, C8 to C2, C9 to C3, C10 to C4, C22 to C6, C19 to C7, C2 to C8, C20 to C9, D7 to D2, D5 to D3, D3 to D4, D1 to D5, D2 to D6, D4 to D8, J5 to J3, J2 to J6, J6 to J7, J3 to J8, R17 to R1, R18 to R10, R16 to R11, R15 to R12, R3 to R17, R4 to R18, R1 to R2, R2 to R3, R13 to R4, R9 to R6, R11 to R7, R10 to R8, R8 to R9, U3 to U1, U1 to U2, U7 to U3, U8 to U4, U11 to U5
Connections:
- net VCC is gone; now on net +3V3: J4.4 (Pin_4)
- net +3V3: now also D7.1 (K), J5.1 (Pin_1)
- net CS_SD: now also U8.15 (SD_CS); no longer U8. (SD_SCK)
- net ESP_RX1: now also U6.3 (A2)
- net ESP_RX2: now also U7.3 (A2)
- net ESP_TX1: now also U6.2 (A1)
- net ESP_TX2: now also U7.2 (A1)
- net GND: now also D7.2 (A), J5.12 (Pin_12)
- net LCD_DC: now also U2.8 (GPIO15/U0RTS/ADC2_CH4/XTAL_32K_P); no longer U2.25 (GPIO48/SPICLK_N/SUBSPICLK_N_DIFF)
- net LCD_TIRQ: now also U2.9 (GPIO16/U0CTS/ADC2_CH5/XTAL_32K_N); no longer U2.8 (GPIO15/U0RTS/ADC2_CH4/XTAL_32K_P)
- net MISO: now also U8.17 (SD_MISO); no longer U8. (SD_SCK)
- net MOSI: now also U8.16 (SD_MOSI); no longer U8. (SD_SCK)
- net SCK: now also U8.18 (SD_CLK); no longer U8. (SD_SCK)
- net GPIO45: now reaches U2.26 (GPIO45)
- net GPIO45: now also J5.5 (Pin_5)
- net GPIO35: now reaches U2.28 (SPIIO6/GPIO35/FSPID/SUBSPID)
- net GPIO35: now also J5.2 (Pin_2)
- net GPIO36: now reaches U2.29 (SPIIO7/GPIO36/FSPICLK/SUBSPICLK)
- net GPIO36: now also J5.3 (Pin_3)
- net GPIO37: now reaches U2.30 (SPIDQS/GPIO37/FSPIQ/SUBSPIQ)
- net GPIO37: now also J5.4 (Pin_4)
- net at U5.13 (GP3): now also J5.7 (Pin_7)
- net at U5.14 (GP4): now also J5.8 (Pin_8)
- net at U5.15 (GP5): now also J5.9 (Pin_9)
- net at U5.16 (GP6): now also J5.10 (Pin_10)
- net at U5.17 (GP7): now also J5.11 (Pin_11)
- net VBAT renamed +BATT
- new net GPIO48: J5.6 (Pin_6), U2.25 (GPIO48/SPICLK_N/SUBSPICLK_N_DIFF)
- no-connect marks 17 -> 7
Other:
- note added: "MCU set to 4.2V"
- note added: "On GPS Module, remove regulator and short Vin to Vout Do Not Connect to Module's USB"
- note removed: "On GPS Module, remove regulator and short Vin to Vout"
- moved on the sheet: C1, C10, C17, C18, C5, C6, C7, C8, C9, J2, R1, U3

Commit message: routing initial
Parts:
- C11: footprint Capacitor_SMD:C_0603_1608Metric -> Capacitor_SMD:C_1206_3216Metric
- C16: footprint Capacitor_SMD:C_0603_1608Metric -> Capacitor_SMD:C_0805_2012Metric
- C17: footprint Capacitor_SMD:C_1206_3216Metric -> Capacitor_SMD:C_0805_2012Metric
- C18: value 22u -> 10u; footprint Capacitor_SMD:C_1206_3216Metric -> Capacitor_SMD:C_0805_2012Metric
- C5, C7, C8: footprint Capacitor_SMD:C_1206_3216Metric -> Capacitor_SMD:C_0603_1608Metric
- J7: footprint Connector_Audio:Jack_3.5mm_CUI_SJ2-3593D-SMT_Horizontal -> wc_sys_footprint:SJ-43514-SMT_CUD
- R2, R3: footprint Resistor_SMD:R_1206_3216Metric -> Resistor_SMD:R_0603_1608Metric
- SW2: footprint Button_Switch_THT:Push_E-Switch_KS01Q01 -> Button_Switch_THT:SW_E-Switch_EG2219_DPDT_Angled; symbol Switch:SW_DIP_x01 -> Switch:SW_Push_DPDT
Connections:
- net Vinput: now also SW2.1 (A), SW2.4 (A); no longer SW2.2
- net at D1.1 (K), Q1.2 (S): now also SW2.2 (B), SW2.5 (B); no longer SW2.1
- net D_N: now reaches U1.4 (I/O2)
- net D_P: now reaches U1.6 (I/O1)
- no-connect marks 7 -> 9
Other:
- moved on the sheet: C5, C6
