File: PCB/finalboard/finalboard.kicad_pcb (KiCad board)
At the start: 4 copper layers, 110 x 70 mm, 66 parts, among them J1 USB_C_Receptacle_USB2.0, J2 Conn_01x04, J3 Conn_01x02, J4 Conn_01x04, J5 Conn_02x06_Counter_Clockwise, J6 Conn_01x02, J7 AudioJack4, J8 Conn_01x04, Q1 DMG2301L, Q2 S8550, SW1 SW_DIP_x01, SW2 SW_DIP_x01, U1 USBLC6-2SC6, U2 ESP32-S3-WROOM-1, U3 AMS1117-3.3, U4 MCP73831-2-OT, U5 MCP23008-xSO, U6 PI4ULS5V202, U7 PI4ULS5V202

Commit message: iterations
Parts:
- moved C14 11.7 mm to (96.0, 56.1), turned to -90 degrees
- moved R5 11.4 mm to (105.9, 66.0), turned to 180 degrees
- moved R6 11.2 mm to (105.9, 70.1), turned to 180 degrees
- moved D2 2.54 mm to (95.2, 69.8)
- moved C13 1.61 mm to (106.2, 47.2)
- moved C15 1.48 mm to (106.9, 54.9)
Routing:
- net /LCD_DC: track 0.00 -> 55.6 mm, vias 0 -> 2
- net /ESP_RX1: track 0.00 -> 52.9 mm, vias 0 -> 4
- net /ESP_TX1: track 0.00 -> 52.0 mm, vias 0 -> 4
- net GND: track 86.2 -> 126.2 mm, vias 27 -> 40
- net Net-(J2-Pin_4): track 0.00 -> 33.2 mm
- net Net-(J2-Pin_3): track 0.00 -> 32.8 mm
- net Net-(J2-Pin_2): track 0.00 -> 32.4 mm
- net Net-(J2-Pin_1): track 0.00 -> 31.9 mm
- net Net-(U2-EN): track 0.00 -> 25.3 mm, vias 0 -> 1
- net /ESP_RX2: track 0.00 -> 22.2 mm, vias 0 -> 2
- net /ESP_TX2: track 0.00 -> 21.9 mm, vias 0 -> 2
- net /CA_RX: track 0.00 -> 16.1 mm
- net /ESP_RX0: track 0.00 -> 15.5 mm
- net Net-(D3-K): track 26.1 -> 40.7 mm, vias 1 -> 2
- net /ESP_TX0: track 0.00 -> 14.3 mm
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