File: PCB/finalboard/finalboard.kicad_pcb (KiCad board)
At the start: 4 copper layers, 110 x 70 mm, 66 parts, among them J1 USB_C_Receptacle_USB2.0, J2 Conn_01x04, J3 Conn_01x02, J4 Conn_01x04, J5 Conn_02x06_Counter_Clockwise, J6 Conn_01x02, J7 AudioJack4, J8 Conn_01x04, Q1 DMG2301L, Q2 S8550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

Commit message: pcb made genesis 1.0
pcb made and manufactured
Routing:
- net Net-(U2-GPIO2/TOUCH2/ADC1_CH1): track 0.00 -> 98.7 mm, vias 0 -> 3
- net Net-(U2-GPIO1/TOUCH1/ADC1_CH0): track 0.00 -> 97.7 mm, vias 0 -> 5
- net Net-(J5-Pin_11): track 0.00 -> 70.8 mm, vias 0 -> 2
- net Net-(J5-Pin_9): track 0.00 -> 67.0 mm, vias 0 -> 2
- net Net-(J5-Pin_10): track 0.00 -> 65.7 mm, vias 0 -> 2
- net /GPIO37: track 0.00 -> 59.5 mm, vias 0 -> 3
- net /GPIO36: track 0.00 -> 59.3 mm, vias 0 -> 5
- net Net-(J5-Pin_7): track 0.00 -> 58.7 mm, vias 0 -> 2
- net /GPIO45: track 0.00 -> 58.6 mm, vias 0 -> 2
- net Net-(J5-Pin_8): track 0.00 -> 57.6 mm, vias 0 -> 2
- net /GPIO35: track 0.00 -> 57.2 mm, vias 0 -> 3
- net /GPIO48: track 0.00 -> 51.6 mm, vias 0 -> 2
- net VBUS: track 25.5 -> 66.9 mm, vias 8 -> 12
- net /LCD_BACKLIGHT: track 0.00 -> 36.8 mm, vias 0 -> 2
- net Net-(D3-K): track 40.7 -> 16.1 mm, vias 2 -> 1
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